File: hardware/base/microclem_base.sch (KiCad schematic (older format))
At the start: 81 parts, among them U1 74LS02, U10 74LS74, U11 74LS74, U12 74LS14, U13 74LS08, U14 74LS32, U15 74LS590, U16 74LS163, U17 74LS163, U18 74LS245, U19 74LS590, U2 74LS08, U20 74LS590, U21 74LS138, U22 74LS245, U3 74LS14, U4 74LS08, U5 74LS74, U6 74LS00, U7 74LS08, U8 74LS32, U9 74LS125, X1 CXO_DIP8

Commit message: base: update specific 74 part references
Parts:
- U1: value 74LS02 -> 74AHC02
- U10, U11, U5: value 74LS74 -> 74AHC74
- U12, U3: value 74LS14 -> 74AHC14
- U13, U2, U4, U7: value 74LS08 -> 74AHC08
- U14, U8: value 74LS32 -> 74AHC32
- U15, U19, U20: value 74LS590 -> 74HC590
- U16, U17: value 74LS163 -> 74AC163
- U18, U22: value 74LS245 -> 74AHCT245
- U21: value 74LS138 -> 74AHC138
- U6: value 74LS00 -> 74AHC00
- U9: value 74LS125 -> 74AHCT125

Commit message: label BASE_CLK signal
Connections:
- net BASE_CLK: now reaches U4.1, X1.5 (OUT)
Changed lines of the file:
@@
 Text Notes 800  6700 0    50   ~ 10
 Reset signals
-Text Notes 3650 4350 0    50   ~ 10
+Text Notes 4250 4400 0    50   ~ 10
 Clock generator/divider
 Wire Wire Line
@@
 	1    0    0    -1
 $EndComp
+Text GLabel 3700 4550 1    50   Input ~ 0
+BASE_CLK
+Wire Wire Line
+	3700 4550 3700 4750
+Connection ~ 3700 4750
 Wire Wire Line
 	21150 7600 21950 7600

Commit message: move BASE_CLK signal
Connections:
- net BASE_CLK: now also JPC2.2 (B), U15.11 (CPC), U15.13 (CPR), U4.3; no longer U4.1, X1.5 (OUT)
- new net: U4.1, X1.5 (OUT)
Changed lines of the file:
@@
 Text Notes 800  6700 0    50   ~ 10
 Reset signals
-Text Notes 4250 4400 0    50   ~ 10
+Text Notes 3750 4400 0    50   ~ 10
 Clock generator/divider
 Wire Wire Line
@@
 $EndComp
 Wire Wire Line
-	4300 4850 5450 4850
-Wire Wire Line
 	5250 5400 5400 5400
 Wire Wire Line
@@
 	1    0    0    -1
 $EndComp
-Text GLabel 3700 4550 1    50   Input ~ 0
+Text GLabel 4600 4700 2    50   Input ~ 0
 BASE_CLK
 Wire Wire Line
-	3700 4550 3700 4750
-Connection ~ 3700 4750
+	4300 4700 4300 4850
+Wire Wire Line
+	4300 4850 5450 4850
+Wire Wire Line
+	4600 4700 4300 4700
 Wire Wire Line
 	21150 7600 21950 7600

Commit message: some base board comments
Other:
- note added: "TODO: fix spacing for these caps on the PCB"
- note added: "TODO: remove functionality that's implemented by the backplane (clock gen. etc.)"
Changed lines of the file:
@@
 Wire Bus Line
 	750  1100 750  2750
+Text Notes -4050 5150 0    50   ~ 0
+TODO: remove functionality that's implemented by the backplane (clock gen. etc.)
+Text Notes 11550 10500 0    50   ~ 0
+TODO: fix spacing for these caps on the PCB
 $EndSCHEMATC

Commit message: update schematics for backplane and base to put PHI_2 on the bus
Connections:
- net +5V: no longer CB4.1, R1.1, R2.1, R6.1, U10.10 (~S), U10.4 (~S), U11.4 (~S), U5.10 (~S), X1.8 (Vcc)
- net BASE_CLK: now also CONN1.C31 (31C); no longer JPC2.2 (B), U15.11 (CPC), U15.13 (CPR), U4.3
- net BUS_ACTIVE: no longer U2.1
- net BUS_CLK: no longer U2.9, U3.1, U5.11 (C)
- net GND: no longer CB4.2, CR1.2, CR2.2, JPC1.2 (B), X1.4 (GND)
- net PHI_2: now also CONN1.A28 (28A), CONN1.B28 (28B), U15.11 (CPC), U15.13 (CPR), U9.2; no longer MP1.37 (ϕ0), R3.2, U11.11 (C), U6.10, U7.12, U7.9, U8.8, VIA1.25 (ϕ2)
- net ~BUS_ACTIVE~: no longer U2.4
- net ~RST~: now also U15.10 (~MRC); no longer U3.8
- net at JPC5.2 (B): no longer U15.2 (Q2)
- net at JPC4.2 (B): no longer U15.1 (Q1)
- net at JPC3.2 (B): no longer U15.15 (Q0)
- net at X1.5 (OUT): no longer U4.1
- net at U3.2: no longer U10.3 (C)
- net at U3.4: no longer U11.3 (C)
- net at U3.11: no longer U3.12
- net at U8.10: no longer U2.11
- net at U8.9: no longer U2.8
- net at U15.3 (Q3), U9.5: no longer JPC6.2 (B)
- net at U10.2 (D): no longer U2.3
- net at U10.5 (Q): no longer U5.12 (D)
- net at U5.8 (~Q): no longer U2.5
- net at U5.9 (Q): no longer U2.10
- net at U11.2 (D): no longer U2.6
- net at U11.5 (Q): no longer U10.12 (D)
- net at U10.8 (~Q): no longer U2.2
- net at U10.9 (Q): no longer U2.12
- net RST-unused: no longer names the net of U3.9
- net RST-unused: no longer U3.6
- removed net SYS_CLK: CONN1.A28 (28A), CONN1.B28 (28B), U10.11 (C), U2.13, U3.3, U9.3, U9.6
- removed net ~CLK_RST~: U10.1 (~R), U10.13 (~R), U11.1 (~R), U15.10 (~MRC), U3.10, U4.2, U5.13 (~R)
- removed net ~RST_HDR~: CONN1.C31 (31C), D1.2 (A), D2.2 (A), JPC1.1 (A), R6.2
- new net: CB4.2, X1.4 (GND)
- new net: CB4.1, X1.8 (Vcc)
- new net BOARD_CLK: MP1.37 (ϕ0), R3.2, U11.11 (C), U6.10, U7.12, U7.9, U9.3, U9.6, VIA1.25 (ϕ2)
- now unconnected: CR1.1, CR2.1, D1.1 (K), D2.1 (K), JPC2.1 (A), JPC3.1 (A), JPC4.1 (A), JPC5.1 (A), JPC6.1 (A), R1.2, R2.2, U3.13, U3.5
Other:
- note added: "BASE_CLK - clock signal generated by some reference on the backplane (e.g. XO or 555)\nBUS_CLK - clock signal driven by some bus device\nPHI_2 - effective system clock signal, either BASE_CLK or BUS_CLK depending on if ~BUS_ACTIVE~ is high or low\nBOARD_CLK - the effective clock rate used by this board. This is PHI_2 unless ~CPY~ is low, in which case we use a /16 divided PHI_2"
- note added: "Clock divider for copy clock"
- note removed: "Clock generator/divider"
- note removed: "Clock switcher"
- note removed: "Reset signals"
- note removed: "TODO: fix spacing for these caps on the PCB"
- note removed: "TODO: remove functionality that's implemented by the backplane (clock gen. etc.)"
- note removed: "shorter clock rst pulse s.t. \nclock starts before other ICs"
- moved on the sheet: CB1, CB10, CB17, CB3, CB4, CB5, CB7, CR1, CR2, D1, D2, JPC1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

Commit message: base: relayout WIP
Parts:
- removed CB2, CB27, CB3, CB4, CB5, CB7: 0.1μF, Capacitor_THT:C_Rect_L7.0mm_W3.5mm_P5.00mm, symbol Device:C_Small
- removed CR1, CR2: 1μF, Capacitor_THT:C_Rect_L7.0mm_W3.5mm_P5.00mm, symbol Device:C_Small
- removed D1, D2: DIODE, Diode_THT:D_DO-15_P2.54mm_Vertical_AnodeUp, symbol pspice:DIODE
- removed JPC1: JP_RST, Connector_PinHeader_2.54mm:PinHeader_1x02_P2.54mm_Vertical, symbol Jumper:Jumper_2_Open
- removed JPC2: /1, Connector_PinHeader_2.54mm:PinHeader_1x02_P2.54mm_Vertical, symbol Jumper:Jumper_2_Open
- removed JPC3: /2, Connector_PinHeader_2.54mm:PinHeader_1x02_P2.54mm_Vertical, symbol Jumper:Jumper_2_Open
- removed JPC4: /4, Connector_PinHeader_2.54mm:PinHeader_1x02_P2.54mm_Vertical, symbol Jumper:Jumper_2_Open
- removed JPC5: /8, Connector_PinHeader_2.54mm:PinHeader_1x02_P2.54mm_Vertical, symbol Jumper:Jumper_2_Open
- removed JPC6: /16, Connector_PinHeader_2.54mm:PinHeader_1x02_P2.54mm_Vertical, symbol Jumper:Jumper_2_Open
- removed R1: 1M, Resistor_THT:R_Axial_DIN0207_L6.3mm_D2.5mm_P2.54mm_Vertical, symbol Device:R
- removed R2: 100k, Resistor_THT:R_Axial_DIN0207_L6.3mm_D2.5mm_P2.54mm_Vertical, symbol Device:R
- removed R6: 4.7k, Resistor_THT:R_Axial_DIN0207_L6.3mm_D2.5mm_P2.54mm_Vertical, symbol Device:R
- removed U10, U11: 74AHC74, Package_DIP:DIP-14_W7.62mm_Socket, symbol 74xx:74LS74
- removed U2, U4: 74AHC08, Package_DIP:DIP-14_W7.62mm_Socket, symbol 74xx:74LS08
- removed U3: 74AHC14, Package_DIP:DIP-14_W7.62mm_Socket, symbol 74xx:74LS14
- removed X1: CXO_DIP8, Oscillator:Oscillator_DIP-8, symbol Oscillator:CXO_DIP8
- added LOGO1: Logo_Microclem, graphics:microclem_logo_mask, symbol Graphic:Logo_Open_Hardware_Small
- added LOGO2: Logo_QR_Code, graphics:qr_code, symbol Graphic:Logo_Open_Hardware_Small
- added LOGO3: Logo_Open_Hardware_Small, Symbol:OSHW-Logo2_9.8x8mm_SilkScreen, symbol Graphic:Logo_Open_Hardware_Small
Connections:
- net +5V: now also U5.10 (~S)
- net BOARD_CLK: now also U5.11 (C)
- net CPY: now also U5.8 (~Q)
- net GND: now also U8.10, U8.9
- net ~CPY~: now also U5.9 (Q)
- net ~RST~: now also U5.13 (~R)
- net at R10.2, U20.7 (Q7): now also U5.12 (D)
- no-connect marks 29 -> 27
Other:
- moved on the sheet: CB11, U12D, U5B, U7A, U8C

Commit message: base: slightly simplify and fix schematic
Parts:
- removed unit 6 of U12
Connections:
- net BUS_STATUS_W is gone; now on net GND: U6.9
- net ~PHI_2~ is gone; now on net ~BOARD_CLK~: R4.2, U1.3, U12.2, U14.4, U14.9, U6.12, U8.12, U8.4
- net BOARD_CLK: now also U12.9; no longer U6.10
- net GND: now also U6.10; no longer U12.9, U8.10, U8.9
- net ~BUS_STATUS_W~: now also U8.9
- net at U8.8: now also U5.3 (C)
- net at U6.8: no longer U5.3 (C)
- net ~BOARD_CLK~: now reaches U12.8
- net ~BOARD_CLK~: now also U8.10
- no-connect marks 27 -> 26
Other:
- note added: "When BOARD_CLK goes low,\nR~W~ goes low for about 220ns\n\nAs the 590 counts on a +ve edge, \nthis gives us set up time for the copy"
- note added: "~BOARD_CLK~ is delayed relative to \nBOARD_CLK by about 12-14ns in testing"
- note removed: "TODO: double check"
- note removed: "TODO: this could be \nOR(~BUS_STATUS_W~, ~PHI_2~)\nif we found a spare OR gate"
- note removed: "When PHI_2 goes low,\nR~W~ goes low for about 220ns\n\nAs the 590 counts on a +ve edge, \nthis gives us set up time for the copy"
- note removed: "~PHI_2~ is delayed relative to \nPHI_2 by about 12-14ns in testing"
- moved on the sheet: U12D, U15, U6C, U7A, U8C, U9A, U9B

Commit message: base: first pass at re-routing
Parts:
- added CB2: 0.1μF, Capacitor_THT:C_Rect_L7.0mm_W3.5mm_P5.00mm, symbol Device:C_Small
- added U2: 74AHC74, Package_DIP:DIP-14_W7.62mm_Socket, symbol 74xx:74LS74
- CR3, CR4: footprint Capacitor_THT:C_Rect_L7.0mm_W3.5mm_P5.00mm -> Capacitor_THT:C_Rect_L10.3mm_W4.5mm_P7.50mm_MKS4
- R10, R11, R3, R4, R5, R7, R8, R9: footprint Resistor_THT:R_Axial_DIN0207_L6.3mm_D2.5mm_P2.54mm_Vertical -> Resistor_THT:R_Axial_DIN0207_L6.3mm_D2.5mm_P7.62mm_Horizontal
Connections:
- net +5V: now also CB2.1, U2.14 (VCC), U2.4 (~S); no longer U5.10 (~S)
- net BOARD_CLK: now also U2.3 (C); no longer U5.11 (C)
- net CPY: now also U2.6 (~Q); no longer U5.8 (~Q)
- net GND: now also U5.10 (~S), U5.11 (C), U5.12 (D), U5.13 (~R), CB2.2, U2.10 (~S), U2.11 (C), U2.12 (D), U2.13 (~R), U2.7 (GND)
- net ~CPY~: now also U2.5 (Q); no longer U5.9 (Q)
- net ~RST~: now also U2.1 (~R); no longer U5.13 (~R)
- net at R10.2, U20.7 (Q7): now also U2.2 (D); no longer U5.12 (D)
- no-connect marks 26 -> 30
Other:
- moved on the sheet: U12E, U5B, U6C
