File: hardware/front_panel/front_panel.sch (KiCad schematic (older format))
At the start: 6 parts, among them J1 C96ABC, U1 NHD-0420H1Z

Commit message: FP WIP
Parts:
- added D1: LED, LED_THT:LED_D5.0mm, symbol Device:LED
- added H5, H6: MountingHole, rails:m5-close, symbol Mechanical:MountingHole
- added JP1, JP3, JP4, JP5, JP6, JP7, JP8: Conn_02x01, Connector_PinHeader_2.54mm:PinHeader_1x02_P2.54mm_Vertical, symbol Connector_Generic:Conn_02x01
- added JP2, JP9: Conn_01x03_Male, Connector_PinHeader_2.54mm:PinHeader_1x03_P2.54mm_Vertical, symbol Connector:Conn_01x03_Male
- added R1: 100k, Potentiometer_THT:Potentiometer_TT_P0915N, symbol Device:R_Variable
- added RN1: R_Network08, Resistor_THT:R_Array_SIP9, symbol Device:R_Network08
- added SW1, SW5: SW_SPDT, symbol Switch:SW_SPDT
- added SW2, SW6: SW_Push, symbol Switch:SW_Push
- added SW3: SW_SPST, symbol Switch:SW_SPST
- added SW7: SW_DIP_x08, Button_Switch_THT:SW_DIP_SPSTx08_Piano_10.8x21.88mm_W7.62mm_P2.54mm, symbol Switch:SW_DIP_x08
- added SW8: SW_Push_LED, symbol Switch:SW_Push_LED
- added U2: 74HC688, Package_DIP:DIP-20_W7.62mm_Socket, symbol 74xx:74HC688
Connections:
- net GND: now also SW7.1, SW7.2, SW7.3, SW7.4, SW7.5, SW7.6, SW7.7, SW7.8, U2.10 (GND)
- net VCC: now also RN1.1 (common), U2.20 (VCC)
- net bd5: now reaches J1.C24 (24C)
- net bd5: now also U2.13 (P5)
- net bd4: now reaches J1.C25 (25C)
- net bd4: now also U2.11 (P4)
- net bd3: now reaches J1.C26 (26C)
- net bd3: now also U2.8 (P3)
- net bd2: now reaches J1.C27 (27C)
- net bd2: now also U2.6 (P2)
- net bd1: now reaches J1.C28 (28C)
- net bd1: now also U2.4 (P1)
- net bd0: now reaches J1.C29 (29C)
- net bd0: now also U2.2 (P0)
- new net: D1.2 (A), JP6.1 (Pin_1)
- new net: D1.1 (K), JP6.2 (Pin_2)
- new net: JP7.1 (Pin_1), SW8.4 (A)
- new net: JP7.2 (Pin_2), SW8.3 (K)
- new net: JP5.1 (Pin_1), SW8.1
- new net: JP5.2 (Pin_2), SW8.2
- new net: JP8.1 (Pin_1), SW6.2
- new net: JP8.2 (Pin_2), SW6.1
- new net: JP4.1 (Pin_1), SW3.1 (A)
- new net: JP4.2 (Pin_2), SW3.2 (B)
- new net: JP1.1 (Pin_1), R1.1
- new net: JP1.2 (Pin_2), R1.2
- new net: JP3.1 (Pin_1), SW2.2
- new net: JP3.2 (Pin_2), SW2.1
- new net: JP2.1 (Pin_1), SW5.1 (A)
- new net: JP2.2 (Pin_2), SW5.2 (B)
- new net: JP2.3 (Pin_3), SW5.3 (C)
- new net: JP9.1 (Pin_1), SW1.1 (A)
- new net: JP9.2 (Pin_2), SW1.2 (B)
- new net: JP9.3 (Pin_3), SW1.3 (C)
- new net: RN1.6 (R5), SW7.12, U2.12 (R4)
- new net: RN1.7 (R6), SW7.11, U2.14 (R5)
- new net: RN1.8 (R7), SW7.10, U2.16 (R6)
- new net: RN1.9 (R8), SW7.9, U2.18 (R7)
- new net: RN1.2 (R1), SW7.16, U2.3 (R0)
- new net: RN1.3 (R2), SW7.15, U2.5 (R1)
- new net: RN1.4 (R3), SW7.14, U2.7 (R2)
- new net: RN1.5 (R4), SW7.13, U2.9 (R3)
- no-connect marks 0 -> 2
Other:
- note added: "555_ADJ"
- note added: "555_STEP"
- note added: "AST_MONO_SW"
- note added: "Bus dev checker"
- note added: "CLK_EN"
- note added: "CLK_SEL"
- note added: "POWER_LED"
- note added: "POWER_SW"
- note added: "RESET_SW"
- note added: "SB_LED"
- note added: "TODO: maybe just put front-side headers to\nconnect to button/led w/ wires"
- note added: "TODO: maybe use ~RST~ in the comparison\nto block until the computer is initialized"
- moved on the sheet: H1, H2, H3, H4

Commit message: front panel: nhd-0440wh 4x40 panel
Parts:
- removed U1: NHD-0420H1Z, Display:NHD-0420H1Z, symbol Display_Character:NHD-0420H1Z
- added U3: NHD-0440WH, nhd-0040wh:NHD-0040WH, symbol nhd0440wh:NHD-0440WH
Connections:
- net GND: now also U3.13 (VSS)
- net VCC: now also U3.14 (VDD)
Changed lines of the file:
@@
 	2200 -1600 2200 -1500
-$Comp
-L Display_Character:NHD-0420H1Z U1
-U 1 1 620A1A2C
-P 4450 3950
-F 0 "U1" H 4450 3950 50  0000 C CNN
-F 1 "NHD-0420H1Z" H 4450 4200 50  0000 C CNN
-F 2 "Display:NHD-0420H1Z" H 4450 3050 50  0001 C CNN
-F 3 "http://www.newhavendisplay.com/specs/NHD-0420H1Z-FSW-GBW-33V3.pdf" H 4550 3850 50  0001 C CNN
-	1    4450 3950
-	1    0    0    -1
-$EndComp
-$Comp
-L power:VCC #PWR0103
-U 1 1 620A39AB
-P 4450 3150
-F 0 "#PWR0103" H 4450 3000 50  0001 C CNN
-F 1 "VCC" H 4465 3323 50  0000 C CNN
-F 2 "" H 4450 3150 50  0001 C CNN
-F 3 "" H 4450 3150 50  0001 C CNN
-	1    4450 3150
-	1    0    0    -1
-$EndComp
-$Comp
-L power:GND #PWR0104
-U 1 1 620A4244
-P 4450 4750
-F 0 "#PWR0104" H 4450 4500 50  0001 C CNN
-F 1 "GND" H 4455 4577 50  0000 C CNN
-F 2 "" H 4450 4750 50  0001 C CNN
-F 3 "" H 4450 4750 50  0001 C CNN
-	1    4450 4750
-	1    0    0    -1
-$EndComp
 $Comp
 L Mechanical:MountingHole H1
@@
 Wire Wire Line
 	8750 1650 8700 1650
+Text Notes 7550 750  0    50   ~ 0
+TODO: maybe just put front-side headers to\nconnect to button/led w/ wires
+$Comp
+L nhd0440wh:NHD-0440WH U3
+U 1 1 620C5F09
+P 5850 4000
+F 0 "U3" H 6250 4550 50  0000 C CNN
+F 1 "NHD-0440WH" H 6250 4850 50  0000 C CNN
+F 2 "nhd-0040wh:NHD-0040WH" H 5550 4950 50  0001 C CNN
+F 3 "" H 5550 4950 50  0001 C CNN
+	1    5850 4000
+	1    0    0    -1
+$EndComp
+$Comp
+L power:VCC #PWR02
+U 1 1 620C72A1
+P 5800 3100
+F 0 "#PWR02" H 5800 2950 50  0001 C CNN
+F 1 "VCC" H 5815 3273 50  0000 C CNN
+F 2 "" H 5800 3100 50  0001 C CNN
+F 3 "" H 5800 3100 50  0001 C CNN
+	1    5800 3100
+	1    0    0    -1
+$EndComp
+$Comp
+L power:GND #PWR03
+U 1 1 620C9013
+P 5800 4700
+F 0 "#PWR03" H 5800 4450 50  0001 C CNN
+F 1 "GND" H 5805 4527 50  0000 C CNN
+F 2 "" H 5800 4700 50  0001 C CNN
+F 3 "" H 5800 4700 50  0001 C CNN
+	1    5800 4700
+	1    0    0    -1
+$EndComp
 Wire Bus Line
 	1700 5500 1700 7100
 Wire Bus Line
 	8700 3200 8700 3700
-Text Notes 7550 750  0    50   ~ 0
-TODO: maybe just put front-side headers to\nconnect to button/led w/ wires
 $EndSCHEMATC
